Commit message: add some xmls

File: mani_skill/assets/robots/panda/panda_v2.urdf (robot description, URDF)
Before this commit: robot panda, 15 links, 14 joints
Links:
- link panda_hand: geometry collision mesh filename=franka_description/meshes/collision/hand.stl; visual mesh filename=franka_description/meshes/visual/hand_visual.obj
- link panda_leftfinger: geometry collision box size=17.5e-3 15.2e-3 18.5e-3; collision box size=17.5e-3 7e-3 23.5e-3
- link panda_link0: geometry collision mesh filename=franka_description/meshes/collision/link0.stl; visual mesh filename=franka_description/meshes/visual/link0_visual.obj
- link panda_link1: geometry collision mesh filename=franka_description/meshes/collision/link1.stl; visual mesh filename=franka_description/meshes/visual/link1_visual.obj
- link panda_link2: geometry collision mesh filename=franka_description/meshes/collision/link2.stl; visual mesh filename=franka_description/meshes/visual/link2_visual.obj
- link panda_link3: geometry collision mesh filename=franka_description/meshes/collision/link3.stl; visual mesh filename=franka_description/meshes/visual/link3_visual.obj
- link panda_link4: geometry collision mesh filename=franka_description/meshes/collision/link4.stl; visual mesh filename=franka_description/meshes/visual/link4_visual.obj
- link panda_link5: geometry collision mesh filename=franka_description/meshes/collision/link5.stl; visual mesh filename=franka_description/meshes/visual/link5_visual.obj
- link panda_link6: geometry collision mesh filename=franka_description/meshes/collision/link6.stl; visual mesh filename=franka_description/meshes/visual/link6_visual.obj
- link panda_link7: geometry collision mesh filename=franka_description/meshes/collision/link7.stl; visual mesh filename=franka_description/meshes/visual/link7_visual.obj
- link panda_rightfinger: geometry collision box size=17.5e-3 15.2e-3 18.5e-3; collision box size=17.5e-3 7e-3 23.5e-3
